File: electronics/Three_Octave_Sharp/Three_Octave_Sharp.kicad_pcb (KiCad board)
At the start: 2 copper layers, 28.6 x 28.6 mm, 33 parts, among them J1 HRO_TYPE-C-31-M-12, J2 FFC Connector, SW1 Alps_Alpine_SKRP, SW2 Alps_Alpine_SKRP, U1 Raspberry_Pi_RP2040, U2 W25Q64JVXGIQ, U3 AP2112K-3.3, Y1 12MHz

Commit message: Add schematic and PCB design copied from Five Octave
Parts:
- added D1: 1N4148WS, Project_Library:D_SOD-323F, F.Cu at (301.7, 38.1)
- added D10: 1N4148WS, Project_Library:D_SOD-323F, F.Cu at (130.2, 38.1)
- added D11: 1N4148WS, Project_Library:D_SOD-323F, F.Cu at (111.2, 38.1)
- added D12: 1N4148WS, Project_Library:D_SOD-323F, F.Cu at (92.1, 38.1)
- added D13: 1N4148WS, Project_Library:D_SOD-323F, F.Cu at (73.1, 38.1)
- added D14: 1N4148WS, Project_Library:D_SOD-323F, F.Cu at (54.0, 38.1)
- added D15: 1N4148WS, Project_Library:D_SOD-323F, F.Cu at (35.0, 38.1)
- added D16: 1N4148WS, Project_Library:D_SOD-323F, F.Cu at (296.9, 57.1)
- added D17: 1N4148WS, Project_Library:D_SOD-323F, F.Cu at (273.1, 57.1)
- added D18: 1N4148WS, Project_Library:D_SOD-323F, F.Cu at (254.0, 57.1)
- added D19: 1N4148WS, Project_Library:D_SOD-323F, F.Cu at (235.0, 57.1)
- added D2: 1N4148WS, Project_Library:D_SOD-323F, F.Cu at (282.6, 38.1)
- added D20: 1N4148WS, Project_Library:D_SOD-323F, F.Cu at (215.9, 57.1)
- added D21: 1N4148WS, Project_Library:D_SOD-323F, F.Cu at (196.9, 57.1)
- added D22: 1N4148WS, Project_Library:D_SOD-323F, F.Cu at (177.8, 57.1)
- added D23: 1N4148WS, Project_Library:D_SOD-323F, F.Cu at (158.8, 57.1)
- added D24: 1N4148WS, Project_Library:D_SOD-323F, F.Cu at (139.7, 57.1)
- added D25: 1N4148WS, Project_Library:D_SOD-323F, F.Cu at (120.7, 57.1)
- added D26: 1N4148WS, Project_Library:D_SOD-323F, F.Cu at (101.6, 57.1)
- added D27: 1N4148WS, Project_Library:D_SOD-323F, F.Cu at (82.6, 57.1)
- added D28: 1N4148WS, Project_Library:D_SOD-323F, F.Cu at (63.5, 57.1)
- added D29: 1N4148WS, Project_Library:D_SOD-323F, F.Cu at (39.7, 57.1)
- added D3: 1N4148WS, Project_Library:D_SOD-323F, F.Cu at (263.6, 38.1)
- added D30: 1N4148WS, Project_Library:D_SOD-323F, F.Cu at (294.5, 76.2)
- added D31: 1N4148WS, Project_Library:D_SOD-323F, F.Cu at (268.3, 76.2)
- added D32: 1N4148WS, Project_Library:D_SOD-323F, F.Cu at (249.3, 76.2)
- added D33: 1N4148WS, Project_Library:D_SOD-323F, F.Cu at (230.2, 76.2)
- added D34: 1N4148WS, Project_Library:D_SOD-323F, F.Cu at (211.2, 76.2)
- added D35: 1N4148WS, Project_Library:D_SOD-323F, F.Cu at (192.1, 76.2)
- added D36: 1N4148WS, Project_Library:D_SOD-323F, F.Cu at (173.1, 76.2)
- added D37: 1N4148WS, Project_Library:D_SOD-323F, F.Cu at (154.0, 76.2)
- added D38: 1N4148WS, Project_Library:D_SOD-323F, F.Cu at (135.0, 76.2)
- added D39: 1N4148WS, Project_Library:D_SOD-323F, F.Cu at (115.9, 76.2)
- added D4: 1N4148WS, Project_Library:D_SOD-323F, F.Cu at (244.5, 38.1)
- added D40: 1N4148WS, Project_Library:D_SOD-323F, F.Cu at (96.9, 76.2)
- added D41: 1N4148WS, Project_Library:D_SOD-323F, F.Cu at (77.8, 76.2)
- added D42: 1N4148WS, Project_Library:D_SOD-323F, F.Cu at (46.9, 76.2)
- added D43: 1N4148WS, Project_Library:D_SOD-323F, F.Cu at (289.8, 95.2)
- added D44: 1N4148WS, Project_Library:D_SOD-323F, F.Cu at (258.8, 95.2)
- added D45: 1N4148WS, Project_Library:D_SOD-323F, F.Cu at (239.8, 95.2)
- added D46: 1N4148WS, Project_Library:D_SOD-323F, F.Cu at (220.7, 95.2)
- added D47: 1N4148WS, Project_Library:D_SOD-323F, F.Cu at (201.7, 95.2)
- added D48: 1N4148WS, Project_Library:D_SOD-323F, F.Cu at (182.6, 95.2)
- added D49: 1N4148WS, Project_Library:D_SOD-323F, F.Cu at (163.6, 95.2)
- added D5: 1N4148WS, Project_Library:D_SOD-323F, F.Cu at (225.5, 38.1)
- added D50: 1N4148WS, Project_Library:D_SOD-323F, F.Cu at (144.5, 95.2)
- added D51: 1N4148WS, Project_Library:D_SOD-323F, F.Cu at (125.5, 95.2)
- added D52: 1N4148WS, Project_Library:D_SOD-323F, F.Cu at (106.4, 95.2)
- added D53: 1N4148WS, Project_Library:D_SOD-323F, F.Cu at (87.4, 95.2)
- added D54: 1N4148WS, Project_Library:D_SOD-323F, F.Cu at (61.2, 95.2)
- added D55: 1N4148WS, Project_Library:D_SOD-323F, F.Cu at (35.0, 95.2)
- added D56: 1N4148WS, Project_Library:D_SOD-323F, F.Cu at (299.3, 114.3)
- added D57: 1N4148WS, Project_Library:D_SOD-323F, F.Cu at (275.5, 114.3)
- added D58: 1N4148WS, Project_Library:D_SOD-323F, F.Cu at (251.7, 114.3)
- added D59: 1N4148WS, Project_Library:D_SOD-323F, F.Cu at (180.2, 114.3)
- added D6: 1N4148WS, Project_Library:D_SOD-323F, F.Cu at (206.4, 38.1)
- added D60: 1N4148WS, Project_Library:D_SOD-323F, F.Cu at (111.2, 114.3)
- added D61: 1N4148WS, Project_Library:D_SOD-323F, F.Cu at (92.1, 114.3)
- added D7: 1N4148WS, Project_Library:D_SOD-323F, F.Cu at (187.4, 38.1)
- added D8: 1N4148WS, Project_Library:D_SOD-323F, F.Cu at (168.3, 38.1)
- added D9: 1N4148WS, Project_Library:D_SOD-323F, F.Cu at (149.3, 38.1)
- added J3: FFC Connector, Project_Library:JUSHUO_AFC01-S16FCC-00, F.Cu at (152.4, 114.3)
- added REF**: Stabilizer_2u, Project_Library:Stabilizer_2u, F.Cu at (50.0, 76.2)
- added REF**: Stabilizer_2u, Project_Library:Stabilizer_2u, F.Cu at (292.9, 95.2)
- added REF**: Stabilizer_6_25u, Project_Library:Stabilizer_6_25u, F.Cu at (183.4, 114.3)
- added SW1: Key Esc, Project_Library:Hot_Swap_Socket_CPG151101S11, F.Cu at (305.4, 34.3)
- added SW10: Key 9, Project_Library:Hot_Swap_Socket_CPG151101S11, F.Cu at (134.0, 34.3)
- added SW11: Key 0, Project_Library:Hot_Swap_Socket_CPG151101S11, F.Cu at (114.9, 34.3)
- added SW12: Key -, Project_Library:Hot_Swap_Socket_CPG151101S11, F.Cu at (95.9, 34.3)
- added SW13: Key =, Project_Library:Hot_Swap_Socket_CPG151101S11, F.Cu at (76.8, 34.3)
- added SW14: Key \, Project_Library:Hot_Swap_Socket_CPG151101S11, F.Cu at (57.8, 34.3)
- added SW15: Key `, Project_Library:Hot_Swap_Socket_CPG151101S11, F.Cu at (38.7, 34.3)
- added SW16: locked, Project_Library:Hot_Swap_Socket_CPG151101S11, F.Cu at (300.7, 53.3)
- added SW17: Key Q, Project_Library:Hot_Swap_Socket_CPG151101S11, F.Cu at (276.9, 53.3)
- added SW18: locked, Project_Library:Hot_Swap_Socket_CPG151101S11, F.Cu at (257.8, 53.3)
- added SW19: Key E, Project_Library:Hot_Swap_Socket_CPG151101S11, F.Cu at (238.8, 53.3)
- added SW2: Key 1, Project_Library:Hot_Swap_Socket_CPG151101S11, F.Cu at (286.4, 34.3)
- added SW20: Key R, Project_Library:Hot_Swap_Socket_CPG151101S11, F.Cu at (219.7, 53.3)
- added SW21: Key T, Project_Library:Hot_Swap_Socket_CPG151101S11, F.Cu at (200.7, 53.3)
- added SW22: Key Y, Project_Library:Hot_Swap_Socket_CPG151101S11, F.Cu at (181.6, 53.3)
- added SW23: Key U, Project_Library:Hot_Swap_Socket_CPG151101S11, F.Cu at (162.6, 53.3)
- added SW24: Key I, Project_Library:Hot_Swap_Socket_CPG151101S11, F.Cu at (143.5, 53.3)
- added SW25: Key O, Project_Library:Hot_Swap_Socket_CPG151101S11, F.Cu at (124.5, 53.3)
- added SW26: Key P, Project_Library:Hot_Swap_Socket_CPG151101S11, F.Cu at (105.4, 53.3)
- added SW27: Key [, Project_Library:Hot_Swap_Socket_CPG151101S11, F.Cu at (86.4, 53.3)
- added SW28: Key ], Project_Library:Hot_Swap_Socket_CPG151101S11, F.Cu at (67.3, 53.3)
- added SW29: Key BS, Project_Library:Hot_Swap_Socket_CPG151101S11, F.Cu at (43.5, 53.3)
- added SW3: Key 2, Project_Library:Hot_Swap_Socket_CPG151101S11, F.Cu at (267.3, 34.3)
- added SW30: Key Caps, Project_Library:Hot_Swap_Socket_CPG151101S11, F.Cu at (298.3, 72.4)
- added SW31: Key A, Project_Library:Hot_Swap_Socket_CPG151101S11, F.Cu at (272.1, 72.4)
- added SW32: Key S, Project_Library:Hot_Swap_Socket_CPG151101S11, F.Cu at (253.0, 72.4)
- added SW33: Key D, Project_Library:Hot_Swap_Socket_CPG151101S11, F.Cu at (234.0, 72.4)
- added SW34: Key F, Project_Library:Hot_Swap_Socket_CPG151101S11, F.Cu at (214.9, 72.4)
- added SW35: Key G, Project_Library:Hot_Swap_Socket_CPG151101S11, F.Cu at (195.9, 72.4)
- added SW36: Key H, Project_Library:Hot_Swap_Socket_CPG151101S11, F.Cu at (176.8, 72.4)
- added SW37: Key J, Project_Library:Hot_Swap_Socket_CPG151101S11, F.Cu at (157.8, 72.4)
- added SW38: Key K, Project_Library:Hot_Swap_Socket_CPG151101S11, F.Cu at (138.7, 72.4)
- added SW39: Key L, Project_Library:Hot_Swap_Socket_CPG151101S11, F.Cu at (119.7, 72.4)
- added SW4: Key 3, Project_Library:Hot_Swap_Socket_CPG151101S11, F.Cu at (248.3, 34.3)
- added SW40: Key ;, Project_Library:Hot_Swap_Socket_CPG151101S11, F.Cu at (100.6, 72.4)
- added SW41: Key ', Project_Library:Hot_Swap_Socket_CPG151101S11, F.Cu at (81.6, 72.4)
- added SW42: Key Return, Project_Library:Hot_Swap_Socket_CPG151101S11, F.Cu at (50.6, 72.4)
- added SW43: Key Shift, Project_Library:Hot_Swap_Socket_CPG151101S11, F.Cu at (293.5, 91.4)
- added SW44: Key Z, Project_Library:Hot_Swap_Socket_CPG151101S11, F.Cu at (262.6, 91.4)
- added SW45: Key X, Project_Library:Hot_Swap_Socket_CPG151101S11, F.Cu at (243.5, 91.4)
- added SW46: Key C, Project_Library:Hot_Swap_Socket_CPG151101S11, F.Cu at (224.5, 91.4)
- added SW47: Key V, Project_Library:Hot_Swap_Socket_CPG151101S11, F.Cu at (205.4, 91.4)
- added SW48: Key B, Project_Library:Hot_Swap_Socket_CPG151101S11, F.Cu at (186.4, 91.4)
- added SW49: Key N, Project_Library:Hot_Swap_Socket_CPG151101S11, F.Cu at (167.3, 91.4)
- added SW5: Key 4, Project_Library:Hot_Swap_Socket_CPG151101S11, F.Cu at (229.2, 34.3)
- added SW50: Key M, Project_Library:Hot_Swap_Socket_CPG151101S11, F.Cu at (148.3, 91.4)
- added SW51: Key ,, Project_Library:Hot_Swap_Socket_CPG151101S11, F.Cu at (129.2, 91.4)
- added SW52: Key ., Project_Library:Hot_Swap_Socket_CPG151101S11, F.Cu at (110.2, 91.4)
- added SW53: Key /, Project_Library:Hot_Swap_Socket_CPG151101S11, F.Cu at (91.1, 91.4)
- added SW54: Key Shift, Project_Library:Hot_Swap_Socket_CPG151101S11, F.Cu at (64.9, 91.4)
- added SW55: Key Fn, Project_Library:Hot_Swap_Socket_CPG151101S11, F.Cu at (38.7, 91.4)
- added SW56: Key Ctrl, Project_Library:Hot_Swap_Socket_CPG151101S11, F.Cu at (303.1, 110.5)
- added SW57: Key Opt, Project_Library:Hot_Swap_Socket_CPG151101S11, F.Cu at (279.2, 110.5)
- added SW58: Key Cmd, Project_Library:Hot_Swap_Socket_CPG151101S11, F.Cu at (255.4, 110.5)
- added SW59: Key Space, Project_Library:Hot_Swap_Socket_CPG151101S11, F.Cu at (184.0, 110.5)
- added SW6: Key 5, Project_Library:Hot_Swap_Socket_CPG151101S11, F.Cu at (210.2, 34.3)
- added SW60: Key Cmd, Project_Library:Hot_Swap_Socket_CPG151101S11, F.Cu at (114.9, 110.5)
- added SW61: Key MO(1), Project_Library:Hot_Swap_Socket_CPG151101S11, F.Cu at (95.9, 110.5)
- added SW7: Key 6, Project_Library:Hot_Swap_Socket_CPG151101S11, F.Cu at (191.1, 34.3)
- added SW8: Key 7, Project_Library:Hot_Swap_Socket_CPG151101S11, F.Cu at (172.1, 34.3)
- added SW9: Key 8, Project_Library:Hot_Swap_Socket_CPG151101S11, F.Cu at (153.0, 34.3)
- moved C1 150.0 mm to (32.5, 199.3)
- moved C10 150.0 mm to (44.1, 188.8)
- moved C11 150.0 mm to (39.2, 185.6)
- moved C12 150.0 mm to (38.2, 185.6)
- moved C13 150.0 mm to (39.6, 199.2)
- moved C14 150.0 mm to (37.2, 185.6)
- moved C15 150.0 mm to (33.5, 178.7)
- moved C16 150.0 mm to (34.5, 183.7)
- moved C2 150.0 mm to (32.5, 201.0)
- moved C3 150.0 mm to (43.2, 186.5)
- moved C4 150.0 mm to (42.2, 186.5)
- moved C5 150.0 mm to (34.0, 189.8)
- moved C6 150.0 mm to (33.2, 193.8)
- moved C7 150.0 mm to (38.6, 199.2)
- moved C8 150.0 mm to (44.7, 193.8)
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- renumbered SW2 to SW_B1, SW1 to SW_R1
Routing:
- net COL2: track 6.29 -> 415.7 mm, vias 0 -> 18
- net COL0: track 6.37 -> 389.1 mm, vias 0 -> 6
- net COL3: track 5.91 -> 384.1 mm, vias 0 -> 20
- net COL5: track 8.14 -> 383.2 mm, vias 0 -> 16
- net COL6: track 14.7 -> 380.6 mm, vias 2 -> 18
- net COL4: track 7.07 -> 367.5 mm, vias 0 -> 18
- net COL7: track 15.4 -> 370.1 mm, vias 2 -> 20
- net COL1: track 6.33 -> 332.2 mm, vias 0 -> 10
- net ROW4: track 6.08 -> 238.8 mm, vias 0 -> 2
- net ROW3: track 6.08 -> 236.4 mm, vias 0 -> 7
- net ROW0: track 6.21 -> 235.3 mm, vias 0 -> 2
- net ROW2: track 6.12 -> 232.1 mm, vias 0 -> 4
- net ROW5: track 6.12 -> 228.3 mm, vias 0 -> 2
- net ROW6: track 6.16 -> 224.8 mm, vias 0 -> 4
- net ROW1: track 6.16 -> 204.4 mm, vias 0 -> 2
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- added copper zone on B.Cu, net (none)
- added copper zone on F.Cu, net (none)
Other:
- board size 28.6 x 28.6 mm -> 288.6 x 176.2 mm
- board text added: "+202401xx"
- board text added: "0.1.0"
- board text added: "locked"
- board text removed: "+20230821"
- board text removed: "1.0.0"

Commit message: Layout keys on PCB
Parts:
- removed the D1 at (301.7, 38.1)
- removed the D10 at (130.2, 38.1)
- removed the D11 at (111.2, 38.1)
- removed the D12 at (92.1, 38.1)
- removed the D13 at (73.1, 38.1)
- removed the D14 at (54.0, 38.1)
- removed the D15 at (35.0, 38.1)
- removed the D2 at (282.6, 38.1)
- removed the D27 at (82.6, 57.1)
- removed the D28 at (63.5, 57.1)
- removed the D3 at (263.6, 38.1)
- removed the D4 at (244.5, 38.1)
- removed D40, D41, D52, D53, D54, D56: 1N4148WS, Project_Library:D_SOD-323F
- removed the D5 at (225.5, 38.1)
- removed the D6 at (206.4, 38.1)
- removed the D7 at (187.4, 38.1)
- removed the D8 at (168.3, 38.1)
- removed the D9 at (149.3, 38.1)
- removed J2, J3: FFC Connector, Project_Library:JUSHUO_AFC01-S16FCC-00
- removed the SW1 at (305.4, 34.3)
- removed the SW10 at (134.0, 34.3)
- removed the SW11 at (114.9, 34.3)
- removed the SW12 at (95.9, 34.3)
- removed the SW13 at (76.8, 34.3)
- removed the SW14 at (57.8, 34.3)
- removed the SW15 at (38.7, 34.3)
- removed the SW2 at (286.4, 34.3)
- removed the SW27 at (86.4, 53.3)
- removed the SW28 at (67.3, 53.3)
- removed the SW3 at (267.3, 34.3)
- removed the SW4 at (248.3, 34.3)
- removed SW40: Key ;, Project_Library:Hot_Swap_Socket_CPG151101S11
- removed SW41: Key ', Project_Library:Hot_Swap_Socket_CPG151101S11
- removed the SW5 at (229.2, 34.3)
- removed SW52: Key ., Project_Library:Hot_Swap_Socket_CPG151101S11
- removed SW53: Key /, Project_Library:Hot_Swap_Socket_CPG151101S11
- removed SW54: Key Shift, Project_Library:Hot_Swap_Socket_CPG151101S11
- removed SW56: Key Ctrl, Project_Library:Hot_Swap_Socket_CPG151101S11
- removed the SW6 at (210.2, 34.3)
- removed the SW7 at (191.1, 34.3)
- removed the SW8 at (172.1, 34.3)
- removed the SW9 at (153.0, 34.3)
- added REF**: Stabilizer_2u, Project_Library:Stabilizer_2u, F.Cu at (54.8, 76.2)
- REF**: value Stabilizer_6_25u -> Stabilizer_6u; footprint Project_Library:Stabilizer_6_25u -> Project_Library:Stabilizer_6u
- SW1: renamed from SW16; value locked -> Key Tab
- SW3: renamed from SW18; value locked -> Key W
- SW33: renamed from SW55; value Key Fn -> Key Shift
- SW34: renamed from SW57; value Key Opt -> Key Ctrl
- SW37: renamed from SW60; value Key Cmd -> Key Opt
- SW38: renamed from SW61; value Key MO(1) -> Key Fn
- moved REF** 42.6 mm to (254.8, 76.2)
- moved SW14 41.0 mm to (232.7, 61.0), turned to 0 degrees
- moved SW20 41.0 mm to (118.4, 61.0), turned to 0 degrees
- moved SW1 41.0 mm to (261.3, 41.9), turned to 0 degrees
- moved SW13 41.0 mm to (258.9, 61.0), turned to 0 degrees
- moved SW15 41.0 mm to (213.7, 61.0), turned to 0 degrees
- moved SW16 41.0 mm to (194.6, 61.0), turned to 0 degrees
- moved SW17 41.0 mm to (175.6, 61.0), turned to 0 degrees
- moved SW18 41.0 mm to (156.5, 61.0), turned to 0 degrees
- moved SW19 41.0 mm to (137.5, 61.0), turned to 0 degrees
- moved SW2 41.0 mm to (237.5, 41.9), turned to 0 degrees
- moved SW21 41.0 mm to (99.4, 61.0), turned to 0 degrees
- moved SW22 41.0 mm to (80.3, 61.0), turned to 0 degrees
- moved SW3 41.0 mm to (218.4, 41.9), turned to 0 degrees
- moved SW4 41.0 mm to (199.4, 41.9), turned to 0 degrees
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- renumbered D16 to D1, D25 to D10, D26 to D11, D29 to D12, D30 to D13, D31 to D14, D32 to D15, D33 to D16, D34 to D17, D35 to D18, D36 to D19, D17 to D2, D37 to D20, D38 to D21, D39 to D22, D42 to D23, D43 to D24, D44 to D25, D45 to D26, D46 to D27, D47 to D28, D48 to D29, D18 to D3, D49 to D30, D50 to D31, D51 to D32, D55 to D33, D57 to D34, D58 to D35, D59 to D36, D60 to D37, D61 to D38, D19 to D4, D20 to D5, D21 to D6, D22 to D7, D23 to D8, D24 to D9, SW25 to SW10, SW26 to SW11, SW29 to SW12, SW30 to SW13, SW31 to SW14, SW32 to SW15, SW33 to SW16, SW34 to SW17, SW35 to SW18, SW36 to SW19, SW17 to SW2, SW37 to SW20, SW38 to SW21, SW39 to SW22, SW42 to SW23, SW43 to SW24, SW44 to SW25, SW45 to SW26, SW46 to SW27, SW47 to SW28, SW48 to SW29, SW49 to SW30, SW50 to SW31, SW51 to SW32, SW58 to SW35, SW59 to SW36, SW19 to SW4, SW20 to SW5, SW21 to SW6, SW22 to SW7, SW23 to SW8, SW24 to SW9
Connections:
- D1 pad 1: ROW1 -> ROW0
- D10 pad 1: ROW5 -> ROW0
- D11 pad 1: ROW5 -> ROW0
- D12 pad 1: ROW5 -> ROW0
- D13 pad 1: ROW2 -> ROW1
- D14 pad 1: ROW2 -> ROW1
- D15 pad 1: ROW2 -> ROW1
- D16 pad 1: ROW2 -> ROW1
- D17 pad 1: ROW2 -> ROW1
- D18 pad 1: ROW2 -> ROW1
- D19 pad 1: ROW6 -> ROW1
- D2 pad 1: ROW1 -> ROW0
- D20 pad 1: ROW6 -> ROW1
- D21 pad 1: ROW6 -> ROW1
- D22 pad 1: ROW6 -> ROW1
- D23 pad 1: ROW6 -> ROW1
- D24 pad 1: ROW3 -> ROW2
- D27 pad 1: ROW3 -> ROW2
- D28 pad 1: ROW3 -> ROW2
- D29 pad 1: ROW3 -> ROW2
- D3 pad 1: ROW1 -> ROW0
- D30 pad 1: ROW7 -> ROW2
- D31 pad 1: ROW7 -> ROW2
- D32 pad 1: ROW7 -> ROW2
- D33 pad 1: ROW6 -> ROW2
- D37 pad 1: ROW7 -> ROW3
- D38 pad 1: ROW7 -> ROW3
- D4 pad 1: ROW1 -> ROW0
- D5 pad 1: ROW1 -> ROW0
- D6 pad 1: ROW1 -> ROW0
- D7 pad 1: ROW5 -> ROW0
- D8 pad 1: ROW5 -> ROW0
- D9 pad 1: ROW5 -> ROW0
- SW10 pad 2: COL3 -> COL9
- SW11 pad 2: COL4 -> COL10
- SW12 pad 2: COL7 -> COL11
- SW14 pad 2: COL3 -> COL1
- SW15 pad 2: COL4 -> COL2
- SW16 pad 2: COL5 -> COL3
- SW17 pad 2: COL6 -> COL4
- SW18 pad 2: COL7 -> COL5
- SW19 pad 2: COL0 -> COL6
- SW2 pad 2: COL3 -> COL1
- SW20 pad 2: COL1 -> COL7
- SW21 pad 2: COL2 -> COL8
- SW22 pad 2: COL3 -> COL9
- SW23 pad 2: COL6 -> COL10
- SW27 pad 2: COL5 -> COL3
- SW28 pad 2: COL6 -> COL4
- SW29 pad 2: COL7 -> COL5
- SW3 pad 2: COL4 -> COL2
- SW30 pad 2: COL0 -> COL6
- SW31 pad 2: COL1 -> COL7
- SW32 pad 2: COL2 -> COL8
- SW33 pad 2: COL7 -> COL9
- SW34 pad 2: COL2 -> COL0
- SW35 pad 2: COL3 -> COL1
- SW36 pad 2: COL4 -> COL2
- SW37 pad 2: COL6 -> COL3
- SW38 pad 2: COL7 -> COL4
- SW4 pad 2: COL5 -> COL3
- SW5 pad 2: COL6 -> COL4
- SW6 pad 2: COL7 -> COL5
- SW7 pad 2: COL0 -> COL6
- SW8 pad 2: COL1 -> COL7
- SW9 pad 2: COL2 -> COL8
Routing:
- net COL2: track 415.7 -> 6.29 mm, vias 18 -> 0
- net COL0: track 389.1 -> 6.37 mm, vias 6 -> 0
- net COL3: track 384.1 -> 5.91 mm, vias 20 -> 0
- net COL5: track 383.2 -> 8.14 mm, vias 16 -> 0
- net COL6: track 380.6 -> 14.7 mm, vias 18 -> 2
- net COL4: track 367.5 -> 7.07 mm, vias 18 -> 0
- net COL7: track 370.1 -> 15.4 mm, vias 20 -> 2
- net COL1: track 332.2 -> 6.33 mm, vias 10 -> 0
- net ROW4: track 238.8 -> 6.08 mm, vias 2 -> 0
- net ROW3: track 236.4 -> 6.08 mm, vias 7 -> 0
- net ROW0: track 235.3 -> 6.21 mm, vias 2 -> 0
- net ROW2: track 232.1 -> 6.12 mm, vias 4 -> 0
- net ROW5: track 228.3 -> 6.12 mm, vias 2 -> 0
- net ROW6: track 224.8 -> 6.16 mm, vias 4 -> 0
- net ROW1: track 204.4 -> 6.16 mm, vias 2 -> 0
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Other:
- board size 288.6 x 176.2 mm -> 250.5 x 176.2 mm
- board text added: "0.1.0+202401xx"
- board text removed: "locked"

Commit message: WIP: Update schematic and PCB design
Parts:
- moved J1 185.3 mm to (152.4, 32.7)
- moved C15 185.3 mm to (145.9, 31.4)
- moved C16 185.3 mm to (146.9, 36.4)
- moved R7 185.3 mm to (150.4, 36.8)
- moved R8 185.3 mm to (154.4, 36.8)
- moved U3 185.3 mm to (145.4, 33.9)
- moved SW_B1 136.4 mm to (113.2, 88.0), turned to 0 degrees
- moved SW_R1 134.2 mm to (133.6, 102.5)
- moved C1 133.2 mm to (122.1, 100.7)
- moved C10 133.2 mm to (133.6, 90.2)
- moved C11 133.2 mm to (128.8, 87.0)
- moved C12 133.2 mm to (127.8, 87.0)
- moved C13 133.2 mm to (129.2, 100.7)
- moved C14 133.2 mm to (126.8, 87.0)
- moved C2 133.2 mm to (122.1, 102.4)
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Connections:
- SW37 pad 2: COL3 -> COL8
- SW38 pad 2: COL4 -> COL9
- U1 pad 17: COL7 -> unconnected-(U1-GPIO14-Pad17)
- U1 pad 18: COL6 -> unconnected-(U1-GPIO15-Pad18)
- U1 pad 2: unconnected-(U1-GPIO0-Pad2) -> COL11
- U1 pad 27: COL5 -> unconnected-(U1-GPIO16-Pad27)
- U1 pad 28: COL4 -> unconnected-(U1-GPIO17-Pad28)
- U1 pad 29: COL3 -> unconnected-(U1-GPIO18-Pad29)
- U1 pad 3: unconnected-(U1-GPIO1-Pad3) -> COL10
- U1 pad 30: COL2 -> unconnected-(U1-GPIO19-Pad30)
- U1 pad 31: COL1 -> COL5
- U1 pad 32: COL0 -> COL4
- U1 pad 34: ROW7 -> COL3
- U1 pad 35: ROW6 -> COL2
- U1 pad 36: ROW5 -> COL1
- U1 pad 37: ROW4 -> COL0
- U1 pad 4: unconnected-(U1-GPIO2-Pad4) -> COL9
- U1 pad 5: unconnected-(U1-GPIO3-Pad5) -> COL8
- U1 pad 6: unconnected-(U1-GPIO4-Pad6) -> COL7
- U1 pad 7: unconnected-(U1-GPIO5-Pad7) -> COL6
Routing:
- net COL7: track 15.4 -> 0.00 mm, vias 2 -> 0
- net unconnected-(U1-GPIO14-Pad17): track 0.00 -> 15.4 mm, vias 0 -> 2
- net unconnected-(U1-GPIO15-Pad18): track 0.00 -> 14.7 mm, vias 0 -> 2
- net COL6: track 14.7 -> 0.00 mm, vias 2 -> 0
- net +3V3: track 73.1 -> 82.0 mm, vias 5 -> 6
- net unconnected-(U1-GPIO16-Pad27): track 0.00 -> 8.14 mm
- net unconnected-(U1-GPIO17-Pad28): track 0.00 -> 7.07 mm
- net unconnected-(U1-GPIO19-Pad30): track 0.00 -> 6.29 mm
- net ROW7: track 6.21 -> 0.00 mm
- net ROW6: track 6.16 -> 0.00 mm
- net ROW5: track 6.12 -> 0.00 mm
- net ROW4: track 6.08 -> 0.00 mm
- net unconnected-(U1-GPIO18-Pad29): track 0.00 -> 5.91 mm
- net Net-(J1-D+-PadA6): track 5.40 -> 8.95 mm, vias 0 -> 1
- net Net-(D5-A): track 5.41 -> 2.28 mm
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- removed copper zone on B.Cu, net (none)
- removed copper zone on F.Cu, net GND
Other:
- board size 250.5 x 176.2 mm -> 247.7 x 76.2 mm
- board text removed: "+202401xx"
- board text removed: "0.1.0"

Commit message: WIP: Update schematic and PCB design
Parts:
- removed LED1: WS2812C-2020-V1, Project_Library:WS2812C-2020
- removed the REF** at (152.4, 95.2)
- moved R4 6.17 mm to (115.4, 85.4), turned to -90 degrees
- moved SW_B1 1.56 mm to (114.3, 89.2), turned to -90 degrees
- moved Y1 0.40 mm to (125.3, 101.2)
- moved C1 0.40 mm to (122.1, 100.3)
- moved C2 0.40 mm to (122.1, 102.0)
- moved R2 0.40 mm to (126.7, 103.5)
Connections:
- U1 pad 14: NEOPIX_POWER -> unconnected-(U1-GPIO11-Pad14)
- U1 pad 15: NEOPIX -> unconnected-(U1-GPIO12-Pad15)
- U1 pad 2: COL11 -> COL6
- U1 pad 3: COL10 -> COL7
- U1 pad 31: COL5 -> COL0
- U1 pad 32: COL4 -> COL1
- U1 pad 34: COL3 -> COL2
- U1 pad 35: COL2 -> ROW3
- U1 pad 36: COL1 -> COL3
- U1 pad 37: COL0 -> COL4
- U1 pad 38: ROW3 -> COL5
- U1 pad 4: COL9 -> COL8
- U1 pad 5: COL8 -> COL9
- U1 pad 6: COL7 -> COL10
- U1 pad 7: COL6 -> COL11
Routing:
- net ROW1: track 6.16 -> 224.7 mm
- net ROW0: track 6.21 -> 222.5 mm
- net ROW2: track 6.12 -> 208.3 mm
- net COL0: track 6.08 -> 180.2 mm, vias 0 -> 8
- net COL1: track 6.12 -> 156.0 mm, vias 0 -> 8
- net ROW3: track 6.08 -> 141.9 mm
- net COL2: track 6.16 -> 137.1 mm, vias 0 -> 8
- net +3V3: track 82.0 -> 151.9 mm
- net Net-(J1-D+-PadA6): track 8.95 -> 75.5 mm, vias 1 -> 2
- net Net-(J1-D--PadA7): track 8.04 -> 73.6 mm, vias 1 -> 2
- net COL5: track 6.33 -> 66.7 mm, vias 0 -> 6
- net COL3: track 6.21 -> 51.7 mm, vias 0 -> 6
- net COL4: track 6.37 -> 51.7 mm, vias 0 -> 6
- net unconnected-(U1-GPIO14-Pad17): track 15.4 -> 0.00 mm, vias 2 -> 0
- net unconnected-(U1-GPIO15-Pad18): track 14.7 -> 0.00 mm, vias 2 -> 0
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
Commit message: WIP: Update schematic and PCB design
Parts:
- added REF**: Stabilizer_6u, Project_Library:Stabilizer_6u, F.Cu at (152.4, 95.2)
Changed lines of the file:
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@@
     )
+  )
+  (footprint "Project_Library:Stabilizer_6u" (layer "F.Cu")
+    (at 152.4 95.25 180)
+    (fp_text reference "REF**" (at 0 -0.5 180 unlocked) (layer "F.SilkS") hide
+        (effects (font (size 1 1) (thickness 0.1)))
+    )
+    (fp_text value "Stabilizer_6u" (at 0 1 180 unlocked) (layer "F.Fab") hide
+        (effects (font (size 1 1) (thickness 0.15)))
+    )
+    (fp_text user "${REFERENCE}" (at 0 2.5 180 unlocked) (layer "F.Fab") hide
+        (effects (font (size 1 1) (thickness 0.15)))
+    )
+    (fp_rect (start -57.15 -9.525) (end 57.15 9.525)
+      (stroke (width 0.12) (type solid)) (fill none) (layer "F.Fab"))
+    (fp_rect (start -51 -9) (end -44 9)
+      (stroke (width 0.1) (type default)) (fill none) (layer "F.Fab"))
+    (fp_rect (start -7.8 -7.8) (end 7.8 7.8)
+      (stroke (width 0.12) (type solid)) (fill none) (layer "F.Fab"))
+    (fp_rect (start 44 -9) (end 51 9)
+      (stroke (width 0.1) (type default)) (fill none) (layer "F.Fab"))
+    (pad "" np_thru_hole circle (at -47.5 -7 180) (size 3.05 3.05) (drill 3.05) (layers "F&B.Cu" "*.Mask"))
+    (pad "" np_thru_hole circle (at -47.5 8.24 180) (size 4.05 4.05) (drill 4.05) (layers "F&B.Cu" "*.Mask"))
+    (pad "" np_thru_hole circle (at 47.5 -7 180) (size 3.05 3.05) (drill 3.05) (layers "F&B.Cu" "*.Mask"))
+    (pad "" np_thru_hole circle (at 47.5 8.24 180) (size 4.05 4.05) (drill 4.05) (layers "F&B.Cu" "*.Mask"))
   )
   (footprint "Capacitor_SMD:C_0402_1005Metric" (layer "F.Cu")

Commit message: WIP: Update PCB design
Parts:
- removed the REF** at (50.0, 57.1)
- removed the REF** at (254.8, 76.2)
- moved D1 20.5 mm to (250.8, 38.1), turned to -90 degrees
- moved D2 16.0 mm to (231.7, 38.1), turned to -90 degrees
- moved D4 16.0 mm to (193.6, 38.1), turned to -90 degrees
- moved D5 16.0 mm to (174.6, 38.1), turned to -90 degrees
- moved D9 16.0 mm to (98.4, 38.1), turned to -90 degrees
- moved D10 16.0 mm to (79.3, 38.1), turned to -90 degrees
- moved D11 16.0 mm to (60.3, 38.1), turned to -90 degrees
- moved D8 16.0 mm to (117.4, 38.1), turned to -90 degrees
- moved D3 16.0 mm to (212.7, 38.1), turned to -90 degrees
- moved D34 14.3 mm to (234.1, 95.2)
- moved D35 14.3 mm to (210.3, 95.2)
- moved SW1 14.3 mm to (247.0, 41.9)
- moved D24 14.3 mm to (243.6, 76.2)
- moved D36 14.3 mm to (141.2, 95.2)
- moved REF** 14.3 mm to (138.1, 95.2)
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Routing:
- net COL3: track 51.7 -> 112.5 mm, vias 6 -> 4
- net COL8: track 0.00 -> 49.7 mm, vias 0 -> 4
- net COL7: track 0.00 -> 49.7 mm, vias 0 -> 4
- net COL6: track 0.00 -> 49.7 mm, vias 0 -> 6
- net COL4: track 51.7 -> 93.0 mm, vias 6 -> 4
- net COL9: track 0.00 -> 21.9 mm, vias 0 -> 2
- net COL5: track 66.7 -> 51.7 mm
- net ROW0: track 222.5 -> 211.6 mm
- net ROW3: track 141.9 -> 132.4 mm
- net ROW1: track 224.7 -> 215.2 mm
- net COL1: track 156.0 -> 164.3 mm, vias 8 -> 6
- net ROW2: track 208.3 -> 203.5 mm
- net COL0: track 180.2 -> 184.6 mm, vias 8 -> 6
- net Net-(D2-A): track 2.28 -> 5.41 mm
- net Net-(D10-A): track 2.28 -> 5.41 mm
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Other:
- board size 247.7 x 76.2 mm -> 228.6 x 76.2 mm

Commit message: WIP: Update PCB design
Parts:
- moved R4 14.3 mm to (97.5, 96.9)
- moved SW_B1 14.3 mm to (96.4, 100.7)
- moved C11 9.60 mm to (109.8, 88.2)
- moved C12 9.60 mm to (108.8, 88.2)
- moved C14 9.60 mm to (107.8, 88.2)
- moved C5 9.60 mm to (104.5, 92.4)
- moved C6 9.60 mm to (103.7, 96.5)
- moved C8 9.60 mm to (115.2, 96.5)
- moved R1 9.60 mm to (112.0, 100.0)
- moved R3 9.60 mm to (101.2, 86.4)
- moved U1 9.60 mm to (109.5, 95.2)
- moved U2 9.60 mm to (102.6, 89.1)
- moved C3 9.60 mm to (113.8, 89.2)
- moved C4 9.60 mm to (112.8, 89.2)
- moved R5 9.60 mm to (110.8, 89.2)
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Connections:
- U1 pad 30: unconnected-(U1-GPIO19-Pad30) -> ROW0
- U1 pad 31: COL0 -> ROW1
- U1 pad 32: COL1 -> ROW2
- U1 pad 34: COL2 -> unconnected-(U1-GPIO22-Pad34)
- U1 pad 35: ROW3 -> COL0
- U1 pad 36: COL3 -> COL1
- U1 pad 37: COL4 -> COL2
- U1 pad 38: COL5 -> ROW3
- U1 pad 39: ROW2 -> COL3
- U1 pad 40: ROW1 -> COL4
- U1 pad 41: ROW0 -> COL5
Routing:
- net COL10: track 0.00 -> 30.2 mm, vias 0 -> 2
- net ROW0: track 211.6 -> 230.7 mm
- net COL9: track 21.9 -> 38.4 mm
- net COL11: track 0.00 -> 13.8 mm
- net COL5: track 51.7 -> 65.2 mm
- net Net-(J1-D--PadA7): track 73.6 -> 83.9 mm
- net Net-(J1-D+-PadA6): track 75.5 -> 85.5 mm
- net +3V3: track 151.9 -> 160.7 mm
- net COL3: track 112.5 -> 104.0 mm
- net COL4: track 93.0 -> 84.8 mm
- net Net-(U1-XOUT): track 6.39 -> 0.00 mm
- net ROW3: track 132.4 -> 126.7 mm
- net COL2: track 137.1 -> 131.8 mm
- net Net-(U1-XIN): track 7.93 -> 4.67 mm
- net +1V1: track 21.5 -> 18.8 mm
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