File: electronics/Three_Octave_Sharp/Three_Octave_Sharp.kicad_pcb (KiCad board)
At the start: 2 copper layers, 228.6 x 76.2 mm, 109 parts, among them J1 HRO_TYPE-C-31-M-12, SW1 Key Tab, SW10 Key O, SW11 Key P, SW12 Key BS, SW13 Key Caps, SW14 Key A, SW15 Key S, SW16 Key D, SW17 Key F, SW18 Key G, SW19 Key H, SW2 Key Q, SW20 Key J, SW21 Key K, SW22 Key L, SW23 Key Return, SW24 Key Shift, SW25 Key Z, SW26 Key X, SW27 Key C, SW28 Key V, SW29 Key B, SW3 Key W, SW30 Key N, SW31 Key M, SW32 Key ,, SW33 Key Shift, SW34 Key Ctrl, SW35 Key Cmd, SW36 Key Space, SW37 Key Opt, SW38 Key Fn, SW4 Key E, SW5 Key R, SW6 Key T, SW7 Key Y, SW8 Key U, SW9 Key I, U1 Raspberry_Pi_RP2040, U2 W25Q64JVXGIQ, U3 AP2112K-3.3, Y1 12MHz

Commit message: WIP: Update PCB design
Parts:
- moved R4 3.60 mm to (101.1, 96.9)
- moved SW_B1 3.60 mm to (100.0, 100.7)
- moved R3 2.60 mm to (99.1, 87.9), turned to 0 degrees
- moved SW_R1 1.16 mm to (119.1, 100.7)
Connections:
- D37 pad 1: ROW3 -> ROW2
- D38 pad 1: ROW3 -> ROW2
- SW37 pad 2: COL8 -> COL10
- SW38 pad 2: COL9 -> COL11
- SW_R1 pad 1: Net-(U1-RUN) -> GND
- SW_R1 pad 2: ~{RESET} -> unconnected-(SW_R1-Pad2)
- SW_R1 pad 3: GND -> Net-(U1-RUN)
- SW_R1 pad 4: unconnected-(SW_R1-Pad4) -> ~{RESET}
- U1 pad 2: COL6 -> COL7
- U1 pad 3: COL7 -> COL8
- U1 pad 32: ROW2 -> unconnected-(U1-GPIO21-Pad32)
- U1 pad 34: unconnected-(U1-GPIO22-Pad34) -> COL0
- U1 pad 35: COL0 -> COL1
- U1 pad 36: COL1 -> COL2
- U1 pad 37: COL2 -> ROW3
- U1 pad 38: ROW3 -> COL3
- U1 pad 39: COL3 -> COL4
- U1 pad 4: COL8 -> COL9
- U1 pad 40: COL4 -> COL5
- U1 pad 41: COL5 -> COL6
- U1 pad 5: COL9 -> ROW2
Routing:
- net COL11: track 13.8 -> 142.6 mm, vias 0 -> 2
- net COL10: track 30.2 -> 158.1 mm, vias 2 -> 4
- net COL9: track 38.4 -> 142.1 mm, vias 2 -> 4
- net ROW2: track 203.9 -> 293.4 mm, vias 0 -> 2
- net COL8: track 49.7 -> 98.3 mm
- net COL7: track 49.7 -> 79.0 mm
- net COL6: track 49.7 -> 73.0 mm
- net COL5: track 65.2 -> 83.2 mm
- net COL3: track 104.0 -> 121.6 mm
- net COL4: track 84.8 -> 102.2 mm
- net COL0: track 186.4 -> 202.4 mm
- net COL2: track 131.8 -> 145.4 mm
- net COL1: track 166.2 -> 173.4 mm
- net Net-(U1-RUN): track 3.11 -> 9.95 mm
- net QSPI_SS_N: track 14.8 -> 19.1 mm, vias 0 -> 2
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
Commit message: WIP: Update PCB design
Parts:
- moved D1 1.20 mm to (250.8, 36.9)
- moved D10 1.20 mm to (79.3, 36.9)
- moved D11 1.20 mm to (60.3, 36.9)
- moved D12 1.20 mm to (41.2, 36.9)
- moved D2 1.20 mm to (231.7, 36.9)
- moved D3 1.20 mm to (212.7, 36.9)
- moved D4 1.20 mm to (193.6, 36.9)
- moved D5 1.20 mm to (174.6, 36.9)
- moved D8 1.20 mm to (117.4, 36.9)
- moved D9 1.20 mm to (98.4, 36.9)
- moved D22 1.20 mm to (74.6, 56.0)
- moved D23 1.20 mm to (48.4, 56.0)
Connections:
- U1 pad 30: ROW0 -> unconnected-(U1-GPIO19-Pad30)
- U1 pad 31: ROW1 -> ROW0
- U1 pad 32: unconnected-(U1-GPIO21-Pad32) -> ROW1
Routing:
- net ROW0: track 229.6 -> 453.9 mm
- net ROW1: track 215.3 -> 417.9 mm
- net Net-(D22-A): track 5.41 -> 0.00 mm
- net unconnected-(U1-GPIO21-Pad32): track 3.82 -> 0.00 mm
- net COL10: track 158.1 -> 157.2 mm, vias 4 -> 2
- net Net-(D3-A): track 5.41 -> 5.94 mm
- net Net-(D12-A): track 5.41 -> 5.94 mm
- net Net-(D5-A): track 5.41 -> 5.94 mm
- net Net-(D4-A): track 5.41 -> 5.94 mm
- net Net-(D1-A): track 5.41 -> 5.94 mm
- net Net-(D8-A): track 5.41 -> 5.94 mm
- net Net-(D23-A): track 5.41 -> 5.94 mm
- net Net-(D9-A): track 5.41 -> 5.94 mm
- net Net-(D11-A): track 5.41 -> 5.94 mm
- net Net-(D10-A): track 5.41 -> 5.94 mm
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
Commit message: WIP: Update PCB design
Parts:
- moved D24 1.20 mm to (243.6, 75.0)
- moved D25 1.20 mm to (217.4, 75.0)
- moved D26 1.20 mm to (198.4, 75.0)
- moved D27 1.20 mm to (179.3, 75.0)
- moved D28 1.20 mm to (160.3, 75.0)
- moved D29 1.20 mm to (141.2, 75.0)
- moved D30 1.20 mm to (122.2, 75.0)
- moved D31 1.20 mm to (103.1, 75.0)
- moved D32 1.20 mm to (84.1, 75.0)
- moved D33 1.20 mm to (53.1, 75.0)
- moved D37 1.20 mm to (74.6, 94.0)
- moved D38 1.20 mm to (55.5, 94.0)
- moved D13 1.20 mm to (248.4, 56.0)
- moved D14 1.20 mm to (227.0, 56.0)
- moved D15 1.20 mm to (207.9, 56.0)
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Routing:
- net ROW1: track 417.9 -> 405.5 mm
- net ROW2: track 293.4 -> 285.6 mm, vias 2 -> 0
- net Net-(D22-A): track 0.00 -> 5.94 mm
- net COL8: track 98.3 -> 95.0 mm
- net COL11: track 142.6 -> 139.6 mm, vias 2 -> 0
- net COL0: track 202.7 -> 200.3 mm
- net COL10: track 157.2 -> 158.8 mm, vias 2 -> 4
- net ROW0: track 453.9 -> 452.6 mm
- net COL1: track 173.8 -> 173.1 mm
- net Net-(D16-A): track 5.41 -> 5.94 mm
- net Net-(D13-A): track 5.41 -> 5.94 mm
- net Net-(D29-A): track 5.41 -> 5.94 mm
- net Net-(D20-A): track 5.41 -> 5.94 mm
- net Net-(D32-A): track 5.41 -> 5.94 mm
- net Net-(D19-A): track 5.41 -> 5.94 mm
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
Commit message: WIP: Update PCB design
Parts:
- moved D34 1.20 mm to (234.1, 94.0)
- moved D35 1.20 mm to (210.3, 94.0)
- moved D36 1.20 mm to (141.2, 94.0)
Routing:
- net COL0: track 200.3 -> 208.2 mm
- net ROW1: track 405.5 -> 413.0 mm
- net ROW0: track 452.6 -> 460.0 mm
- net COL1: track 173.1 -> 179.9 mm
- net +3V3: track 163.8 -> 162.4 mm
- net COL5: track 83.1 -> 81.8 mm
- net ROW3: track 122.9 -> 121.7 mm
- net COL2: track 145.3 -> 146.2 mm
- net Net-(J1-D--PadA7): track 82.5 -> 81.7 mm
- net Net-(J1-D+-PadA6): track 84.1 -> 83.5 mm
- net Net-(D36-A): track 5.41 -> 5.94 mm
- net Net-(D35-A): track 5.41 -> 5.94 mm
- net Net-(D34-A): track 5.41 -> 5.94 mm
