File: electronics/Three_Octave_Sharp/Three_Octave_Sharp.kicad_pcb (KiCad board)
At the start: 2 copper layers, 228.6 x 76.2 mm, 109 parts, among them J1 HRO_TYPE-C-31-M-12, SW1 Key Tab, SW10 Key O, SW11 Key P, SW12 Key BS, SW13 Key Caps, SW14 Key A, SW15 Key S, SW16 Key D, SW17 Key F, SW18 Key G, SW19 Key H, SW2 Key Q, SW20 Key J, SW21 Key K, SW22 Key L, SW23 Key Return, SW24 Key Shift, SW25 Key Z, SW26 Key X, SW27 Key C, SW28 Key V, SW29 Key B, SW3 Key W, SW30 Key N, SW31 Key M, SW32 Key ,, SW33 Key Shift, SW34 Key Ctrl, SW35 Key Cmd, SW36 Key Space, SW37 Key Opt, SW38 Key Fn, SW4 Key E, SW5 Key R, SW6 Key T, SW7 Key Y, SW8 Key U, SW9 Key I, U1 Raspberry_Pi_RP2040, U2 W25Q64JVXGIQ, U3 AP2112K-3.3, Y1 12MHz

Commit message: WIP: Update case design
Parts:
- added REF**: MountingHole_2.2mm_M2, MountingHole:MountingHole_2.2mm_M2, F.Cu at (31.1, 102.3)
- added REF**: MountingHole_2.2mm_M2, MountingHole:MountingHole_2.2mm_M2, F.Cu at (254.7, 102.3)
- added REF**: MountingHole_2.2mm_M2, MountingHole:MountingHole_2.2mm_M2, F.Cu at (234.6, 50.1)
- added REF**: MountingHole_2.2mm_M2, MountingHole:MountingHole_2.2mm_M2, F.Cu at (58.3, 50.1)
Routing:
- net ROW0: track 460.0 -> 458.1 mm
- net ROW1: track 413.0 -> 411.5 mm

Commit message: WIP: Update 3d design
Parts:
- moved REF** 42.4 mm to (68.9, 83.2)
- moved REF** 33.3 mm to (227.4, 83.2)
Changed lines of the file:
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@@
   )
   (footprint "MountingHole:MountingHole_2.2mm_M2" (layer "F.Cu")
-    (at 31.075 102.275)
+    (at 68.9375 83.225)
     (descr "Mounting Hole 2.2mm, no annular, M2")
     (tags "mounting hole 2.2mm no annular m2")
@@
   )
   (footprint "MountingHole:MountingHole_2.2mm_M2" (layer "F.Cu")
-    (at 254.675 102.275)
+    (at 227.409375 83.225)
     (descr "Mounting Hole 2.2mm, no annular, M2")
     (tags "mounting hole 2.2mm no annular m2")
@@
   (gr_rect (start 28.575 66.675) (end 71.4375 85.725)
     (stroke (width 0.1) (type default)) (fill none) (layer "F.Fab"))
-  (gr_rect (start 252.175 99.775) (end 257.175 104.775)
-    (stroke (width 0.1) (type default)) (fill none) (layer "F.Fab"))
   (gr_line (start 111.9375 99.425) (end 113.5375 99.425)
     (stroke (width 0.2) (type default)) (layer "F.Fab"))
@@
   (gr_line (start 113.7125 98.25) (end 114.5125 98.25)
     (stroke (width 0.2) (type default)) (layer "F.Fab"))
-  (gr_rect (start 53.04375 47.615) (end 63.6375 52.615)
+  (gr_rect (start 54.76875 47.625) (end 61.9125 52.615)
     (stroke (width 0.1) (type default)) (fill none) (layer "F.Fab"))
   (gr_line (start 104.7625 97.45) (end 105.1625 97.05)
@@
   (gr_line (start 105.3625 97.45) (end 106.1 97.45)
     (stroke (width 0.2) (type default)) (layer "F.Fab"))
-  (gr_rect (start 28.575 99.775) (end 33.575 104.775)
+  (gr_rect (start 66.4375 80.725) (end 71.4375 85.725)
     (stroke (width 0.1) (type default)) (fill none) (layer "F.Fab"))
   (gr_line (start 104.9625 96.65) (end 106.1 96.65)
@@
   (gr_line (start 112.1375 99.025) (end 113.3375 99.025)
     (stroke (width 0.2) (type default)) (layer "F.Fab"))
+  (gr_rect (start 223.8375 80.725) (end 230.98125 85.725)
+    (stroke (width 0.1) (type default)) (fill none) (layer "F.Fab"))
   (gr_line (start 111.7375 99.225) (end 111.7375 98.6875)
     (stroke (width 0.2) (type default)) (layer "F.Fab"))

Commit message: Rename
Parts:
- added REF**: Fiducial_1mm_Mask2mm, Fiducial:Fiducial_1mm_Mask2mm, F.Cu at (253.2, 24.6)
- added REF**: Fiducial_1mm_Mask2mm, Fiducial:Fiducial_1mm_Mask2mm, F.Cu at (32.6, 108.8)
- added REF**: Fiducial_1mm_Mask2mm, Fiducial:Fiducial_1mm_Mask2mm, F.Cu at (32.6, 24.6)
- added REF**: Fiducial_1mm_Mask2mm, Fiducial:Fiducial_1mm_Mask2mm, F.Cu at (253.2, 108.8)
Other:
- board size 228.6 x 76.2 mm -> 228.6 x 92.2 mm

Commit message: Update PCB version number
Other:
- board text added: "1.0.0+20240125"
- board text removed: "0.1.0+202401xx"
Changed lines of the file:
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@@
   (paper "A4")
   (title_block
-    (title "Three Octave #")
-    (date "2024-01-xx")
-    (rev "0.1.0")
+    (title "Three Octave Sharp")
+    (date "2024-01-25")
+    (rev "1.0.0")
     (comment 1 "https://github.com/takayoshiotake/three-octave-sharp-38-key-keyboard")
   )
@@
     (effects (font (size 1 1) (thickness 0.15)) (justify bottom))
   )
-  (gr_text "0.1.0+202401xx" (at 160.6625 100.0625) (layer "F.SilkS")
+  (gr_text "1.0.0+20240125" (at 160.6625 100.0625) (layer "F.SilkS")
     (effects (font (size 1 1) (thickness 0.15)) (justify left))
   )

Commit message: Fix pcb outline (0.005 mm)
Other:
- board text added: "1.0.1+20240211"
- board text removed: "1.0.0+20240125"
Changed lines of the file:
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@@
     )
     (stroke (width 0) (type solid)) (fill solid) (layer "F.Mask"))
-  (gr_circle (center 38.5 26.87) (end 38.5 27.17)
-    (stroke (width 0.1) (type solid)) (fill none) (layer "Edge.Cuts"))
-  (gr_arc (start 35.5 28.27) (mid 35.412132 28.482132) (end 35.2 28.57)
-    (stroke (width 0.1) (type solid)) (layer "Edge.Cuts"))
-  (gr_line (start 40.7 26.87) (end 40.7 28.27)
+  (gr_circle (center 38.5 26.875) (end 38.5 27.175)
+    (stroke (width 0.1) (type solid)) (fill none) (layer "Edge.Cuts"))
+  (gr_arc (start 35.5 28.275) (mid 35.412132 28.487132) (end 35.2 28.575)
+    (stroke (width 0.1) (type solid)) (layer "Edge.Cuts"))
+  (gr_line (start 40.7 26.875) (end 40.7 28.275)
     (stroke (width 0.1) (type solid)) (layer "Edge.Cuts"))
   (gr_arc (start 250.25 26.875) (mid 250.337868 26.662868) (end 250.55 26.575)
@@
   (gr_line (start 242.66875 106.475) (end 242.66875 105.075)
     (stroke (width 0.1) (type solid)) (layer "Edge.Cuts"))
-  (gr_line (start 28.575 26.57) (end 28.575 20.57)
+  (gr_line (start 28.575 26.575) (end 28.575 20.575)
     (stroke (width 0.1) (type default)) (layer "Edge.Cuts"))
   (gr_arc (start 242.36875 104.775) (mid 242.580857 104.862893) (end 242.66875 105.075)
     (stroke (width 0.1) (type solid)) (layer "Edge.Cuts"))
-  (gr_line (start 29.575 28.57) (end 35.2 28.57)
+  (gr_line (start 29.575 28.575) (end 35.2 28.575)
     (stroke (width 0.1) (type default)) (layer "Edge.Cuts"))
   (gr_circle (center 244.86875 106.475) (end 244.86875 106.175)
     (stroke (width 0.1) (type solid)) (fill none) (layer "Edge.Cuts"))
-  (gr_line (start 35.2 26.57) (end 28.575 26.57)
+  (gr_line (start 35.2 26.575) (end 28.575 26.575)
     (stroke (width 0.1) (type default)) (layer "Edge.Cuts"))
   (gr_line (start 35.5 106.475) (end 35.5 105.075)
@@
   (gr_arc (start 244.75 26.575) (mid 244.962132 26.662868) (end 245.05 26.875)
     (stroke (width 0.1) (type solid)) (layer "Edge.Cuts"))
-  (gr_circle (center 36.1 28.27) (end 36.1 28.57)
+  (gr_circle (center 36.1 28.275) (end 36.1 28.575)
     (stroke (width 0.1) (type solid)) (fill none) (layer "Edge.Cuts"))
   (gr_circle (center 244.06875 106.475) (end 244.06875 106.175)
@@
   (gr_arc (start 247.86875 105.075) (mid 247.956607 104.862857) (end 248.16875 104.775)
     (stroke (width 0.1) (type solid)) (layer "Edge.Cuts"))
-  (gr_circle (center 36.9 26.87) (end 36.9 27.17)
+  (gr_circle (center 36.9 26.875) (end 36.9 27.175)
     (stroke (width 0.1) (type solid)) (fill none) (layer "Edge.Cuts"))
   (gr_circle (center 249.65 28.275) (end 249.65 28.575)
@@
   (gr_circle (center 245.65 28.275) (end 245.65 28.575)
     (stroke (width 0.1) (type solid)) (fill none) (layer "Edge.Cuts"))
-  (gr_arc (start 35.2 26.57) (mid 35.412103 26.657897) (end 35.5 26.87)
-    (stroke (width 0.1) (type solid)) (layer "Edge.Cuts"))
-  (gr_circle (center 37.7 26.87) (end 37.7 27.17)
-    (stroke (width 0.1) (type solid)) (fill none) (layer "Edge.Cuts"))
-  (gr_circle (center 40.1 26.87) (end 40.1 27.17)
+  (gr_arc (start 35.2 26.575) (mid 35.412103 26.662897) (end 35.5 26.875)
+    (stroke (width 0.1) (type solid)) (layer "Edge.Cuts"))
+  (gr_circle (center 37.7 26.875) (end 37.7 27.175)
+    (stroke (width 0.1) (type solid)) (fill none) (layer "Edge.Cuts"))
+  (gr_circle (center 40.1 26.875) (end 40.1 27.175)
     (stroke (width 0.1) (type solid)) (fill none) (layer "Edge.Cuts"))
   (gr_circle (center 38.5 105.075) (end 38.5 104.775)
     (stroke (width 0.1) (type solid)) (fill none) (layer "Edge.Cuts"))
-  (gr_line (start 244.75 26.575) (end 41 26.57)
+  (gr_line (start 244.75 26.575) (end 41 26.575)
     (stroke (width 0.1) (type default)) (layer "Edge.Cuts"))
   (gr_arc (start 29.575 104.775) (mid 28.867894 104.482107) (end 28.575 103.775)
@@
   (gr_circle (center 36.9 106.475) (end 36.9 106.175)
     (stroke (width 0.1) (type solid)) (fill none) (layer "Edge.Cuts"))
-  (gr_line (start 28.575 20.57) (end 257.175 20.575)
+  (gr_line (start 28.575 20.575) (end 257.175 20.575)
     (stroke (width 0.1) (type default)) (layer "Edge.Cuts"))
   (gr_line (start 256.175 104.775) (end 248.16875 104.775)
     (stroke (width 0.1) (type default)) (layer "Edge.Cuts"))
-  (gr_line (start 41 28.57) (end 244.75 28.575)
+  (gr_line (start 41 28.575) (end 244.75 28.575)
     (stroke (width 0.1) (type default)) (layer "Edge.Cuts"))
   (gr_circle (center 39.3 106.475) (end 39.3 106.175)
@@
   (gr_line (start 247.86875 105.075) (end 247.86875 106.475)
     (stroke (width 0.1) (type solid)) (layer "Edge.Cuts"))
-  (gr_circle (center 40.1 28.27) (end 40.1 28.57)
+  (gr_circle (center 40.1 28.275) (end 40.1 28.575)
     (stroke (width 0.1) (type solid)) (fill none) (layer "Edge.Cuts"))
   (gr_circle (center 247.25 28.275) (end 247.25 28.575)
@@
   (gr_circle (center 37.7 106.475) (end 37.7 106.175)
     (stroke (width 0.1) (type solid)) (fill none) (layer "Edge.Cuts"))
-  (gr_line (start 35.5 28.27) (end 35.5 26.87)
+  (gr_line (start 35.5 28.275) (end 35.5 26.875)
     (stroke (width 0.1) (type solid)) (layer "Edge.Cuts"))
   (gr_line (start 257.175 112.775) (end 28.575 112.775)
@@
   (gr_circle (center 247.26875 106.475) (end 247.26875 106.175)
     (stroke (width 0.1) (type solid)) (fill none) (layer "Edge.Cuts"))
-  (gr_arc (start 41 28.57) (mid 40.787897 28.482103) (end 40.7 28.27)
+  (gr_arc (start 41 28.575) (mid 40.787897 28.487103) (end 40.7 28.275)
     (stroke (width 0.1) (type solid)) (layer "Edge.Cuts"))
   (gr_arc (start 250.55 28.575) (mid 250.337868 28.487132) (end 250.25 28.275)
@@
   (gr_circle (center 243.26875 105.075) (end 243.26875 104.775)
     (stroke (width 0.1) (type solid)) (fill none) (layer "Edge.Cuts"))
-  (gr_circle (center 39.3 28.27) (end 39.3 28.57)
+  (gr_circle (center 39.3 28.275) (end 39.3 28.575)
     (stroke (width 0.1) (type solid)) (fill none) (layer "Edge.Cuts"))
   (gr_line (start 257.175 106.775) (end 257.175 112.775)
@@
   (gr_line (start 40.7 105.075) (end 40.7 106.475)
     (stroke (width 0.1) (type solid)) (layer "Edge.Cuts"))
-  (gr_circle (center 36.9 28.27) (end 36.9 28.57)
+  (gr_circle (center 36.9 28.275) (end 36.9 28.575)
     (stroke (width 0.1) (type solid)) (fill none) (layer "Edge.Cuts"))
   (gr_line (start 257.175 26.575) (end 257.175 20.575)
@@
   (gr_line (start 257.175 29.575) (end 257.175 103.775)
     (stroke (width 0.1) (type default)) (layer "Edge.Cuts"))
-  (gr_circle (center 37.7 28.27) (end 37.7 28.57)
+  (gr_circle (center 37.7 28.275) (end 37.7 28.575)
     (stroke (width 0.1) (type solid)) (fill none) (layer "Edge.Cuts"))
   (gr_circle (center 248.85 26.875) (end 248.85 27.175)
@@
   (gr_arc (start 256.175 28.575) (mid 256.882107 28.867893) (end 257.175 29.575)
     (stroke (width 0.1) (type default)) (layer "Edge.Cuts"))
-  (gr_circle (center 38.5 28.27) (end 38.5 28.57)
+  (gr_circle (center 38.5 28.275) (end 38.5 28.575)
     (stroke (width 0.1) (type solid)) (fill none) (layer "Edge.Cuts"))
   (gr_circle (center 247.26875 105.075) (end 247.26875 104.775)
@@
   (gr_circle (center 243.26875 106.475) (end 243.26875 106.175)
     (stroke (width 0.1) (type solid)) (fill none) (layer "Edge.Cuts"))
-  (gr_arc (start 40.7 26.87) (mid 40.787868 26.657868) (end 41 26.57)
+  (gr_arc (start 40.7 26.875) (mid 40.787868 26.662868) (end 41 26.575)
     (stroke (width 0.1) (type solid)) (layer "Edge.Cuts"))
   (gr_arc (start 245.05 28.275) (mid 244.962132 28.487132) (end 244.75 28.575)
     (stroke (width 0.1) (type solid)) (layer "Edge.Cuts"))
-  (gr_circle (center 36.1 26.87) (end 36.1 27.17)
+  (gr_circle (center 36.1 26.875) (end 36.1 27.175)
     (stroke (width 0.1) (type solid)) (fill none) (layer "Edge.Cuts"))
   (gr_circle (center 248.05 26.875) (end 248.05 27.175)
@@
   (gr_circle (center 246.46875 105.075) (end 246.46875 104.775)
     (stroke (width 0.1) (type solid)) (fill none) (layer "Edge.Cuts"))
-  (gr_circle (center 39.3 26.87) (end 39.3 27.17)
+  (gr_circle (center 39.3 26.875) (end 39.3 27.175)
     (stroke (width 0.1) (type solid)) (fill none) (layer "Edge.Cuts"))
   (gr_arc (start 35.2 104.775) (mid 35.412132 104.862868) (end 35.5 105.075)
@@
     (effects (font (size 1 1) (thickness 0.15)) (justify bottom))
   )
-  (gr_text "1.0.0+20240125" (at 160.6625 100.0625) (layer "F.SilkS")
+  (gr_text "1.0.1+20240211" (at 160.6625 100.0625) (layer "F.SilkS")
     (effects (font (size 1 1) (thickness 0.15)) (justify left))
   )
@@
     (polygon
       (pts
-        (xy 35.2 28.77)
-        (xy 35.2 26.37)
-        (xy 41 26.37)
-        (xy 41 28.77)
+        (xy 35.2 28.775)
+        (xy 35.2 26.375)
+        (xy 41 26.375)
+        (xy 41 28.775)
       )
     )
