File: electronics/Three_Octave_Sharp/Three_Octave_Sharp.kicad_sch (KiCad schematic)
At the start: 107 parts, among them J1 HRO_TYPE-C-31-M-12, SW1 Key Tab, SW10 Key O, SW11 Key P, SW12 Key BS, SW16 Key Caps, SW17 Key A, SW18 Key S, SW19 Key D, SW2 Key Q, SW20 Key F, SW21 Alps_Alpine_SKRP, SW21 Key G, SW22 Alps_Alpine_SKRP, SW22 Key H, SW23 Key J, SW24 Key K, SW25 Key L, SW26 Key Return, SW3 Key W, SW30 Key Shift, SW31 Key Z, SW32 Key X, SW33 Key C, SW33 Key Shift, SW34 Key V, SW35 Key B, SW36 Key N, SW37 Key M, SW38 Key ,, SW4 Key E, SW43 Key Ctrl, SW44 Key Cmd, SW45 Key Space, SW46 Key Opt, SW47 Key Fn, SW5 Key R, SW6 Key T, SW7 Key Y, SW8 Key U, SW9 Key I, U1 AP2112K-3.3, U2 Raspberry_Pi_RP2040, U2 W25Q64JVXGIQ, Y1 12MHz

Commit message: Change resistor part # for JLCPCB
Parts:
- R3, R4: LCSC C352446 -> C25100
Changed lines of the file:
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@@
       (effects (font (size 1.27 1.27)) hide)
     )
-    (property "LCSC" "C352446" (at 57.785 157.48 0)
+    (property "LCSC" "C25100" (at 57.785 157.48 0)
       (effects (font (size 1.27 1.27)) hide)
     )
@@
       (effects (font (size 1.27 1.27)) hide)
     )
-    (property "LCSC" "C352446" (at 52.705 152.4 0)
-      (effects (font (size 1.27 1.27)) hide)
-    )
+    (property "LCSC" "C25100" (at 52.705 152.4 0)
+      (effects (font (size 1.27 1.27)) hide)
+    )

Commit message: Update PCB version number
Other:
- title: Three Octave # -> Three Octave Sharp
Changed lines of the file:
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@@
   (paper "A3")
   (title_block
-    (title "Three Octave #")
-    (date "2024-01-xx")
-    (rev "0.1.0")
+    (title "Three Octave Sharp")
+    (date "2024-01-25")
+    (rev "1.0.0")
     (comment 1 "https://github.com/takayoshiotake/three-octave-sharp-38-key-keyboard")
   )
