File: electronics/Three_Octave_Sharp/Three_Octave_Sharp_Simple.kicad_pcb (KiCad board)
At the start: 2 copper layers, 228.6 x 92.2 mm, 117 parts, among them J1 HRO_TYPE-C-31-M-12, SW1 Key Tab, SW10 Key O, SW11 Key P, SW12 Key BS, SW13 Key Caps, SW14 Key A, SW15 Key S, SW16 Key D, SW17 Key F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

Commit message: Rename
Parts:
- removed the REF** at (253.2, 24.6)
- removed the REF** at (32.6, 108.8)
- removed the REF** at (32.6, 24.6)
- removed the REF** at (253.2, 108.8)
Other:
- board size 228.6 x 92.2 mm -> 228.6 x 76.2 mm
